File: hardware/NOT/logicBlocks-NOT.brd (EAGLE design)
At the start: 15.2 x 23.4 mm, 14 parts, among them U1 INVERTER""

Commit message: changed to regular fiducials
Parts:
- removed JP3, JP5, JP6, JP7: FIDUCIALUFIDUCIAL, SparkFun:MICRO-FIDUCIAL
- added FID1, FID2, FID3, FID4: FIDUCIAL1X2, SparkFun-Aesthetics:FIDUCIAL-1X2
