File: hardware/NOT/logicBlocks-NOT.sch (EAGLE design)
At the start: 14 parts, among them U1 INVERTER""

Commit message: changed to regular fiducials
Parts:
- removed JP3, JP5, JP6, JP7: FIDUCIALUFIDUCIAL, SparkFun:FIDUCIALUFIDUCIAL
- added FID1, FID2, FID3, FID4: FIDUCIAL1X2, SparkFun-Aesthetics:FIDUCIAL1X2
Changed lines of the file:
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@@
 <?xml version="1.0" encoding="utf-8"?>
 <!DOCTYPE eagle SYSTEM "eagle.dtd">
-<eagle version="6.2">
+<eagle version="6.6.0">
 <drawing>
 <settings>
@@
 <layer number="106" name="bPlate" color="7" fill="1" visible="yes" active="yes"/>
 <layer number="107" name="Crop" color="7" fill="1" visible="yes" active="yes"/>
+<layer number="108" name="tplace-old" color="10" fill="1" visible="no" active="yes"/>
+<layer number="109" name="ref-old" color="11" fill="1" visible="no" active="yes"/>
 <layer number="116" name="Patch_BOT" color="9" fill="4" visible="yes" active="yes"/>
 <layer number="121" name="_tsilk" color="7" fill="1" visible="yes" active="yes"/>
@@
 <part name="C2" library="SparkFun" deviceset="CAP" device="0402-CAP" value="1uF"/>
 <part name="GND6" library="SparkFun" deviceset="GND" device=""/>
-<part name="JP3" library="SparkFun" deviceset="FIDUCIAL" device="UFIDUCIAL"/>
-<part name="JP5" library="SparkFun" deviceset="FIDUCIAL" device="UFIDUCIAL"/>
-<part name="JP6" library="SparkFun" deviceset="FIDUCIAL" device="UFIDUCIAL"/>
-<part name="JP7" library="SparkFun" deviceset="FIDUCIAL" device="UFIDUCIAL"/>
 <part name="JP8" library="SparkFun-Connectors" deviceset="M03" device="SMD_RA_MALE_POST" value="OUTPUT"/>
+<part name="FID1" library="SparkFun-Aesthetics" deviceset="FIDUCIAL" device="1X2"/>
+<part name="FID2" library="SparkFun-Aesthetics" deviceset="FIDUCIAL" device="1X2"/>
+<part name="FID3" library="SparkFun-Aesthetics" deviceset="FIDUCIAL" device="1X2"/>
+<part name="FID4" library="SparkFun-Aesthetics" deviceset="FIDUCIAL" device="1X2"/>
 </parts>
 <sheets>
@@
 <instance part="C2" gate="G$1" x="149.86" y="91.44"/>
 <instance part="GND6" gate="1" x="149.86" y="71.12"/>
-<instance part="JP3" gate="G$1" x="154.94" y="30.48"/>
-<instance part="JP5" gate="G$1" x="162.56" y="30.48"/>
-<instance part="JP6" gate="G$1" x="162.56" y="25.4"/>
-<instance part="JP7" gate="G$1" x="154.94" y="25.4"/>
 <instance part="JP8" gate="G$1" x="170.18" y="99.06" rot="R180"/>
+<instance part="FID1" gate="G$1" x="238.76" y="33.02"/>
+<instance part="FID2" gate="G$1" x="243.84" y="33.02"/>
+<instance part="FID3" gate="G$1" x="243.84" y="27.94"/>
+<instance part="FID4" gate="G$1" x="238.76" y="27.94"/>
 </instances>
 <busses>
